File: sop8breakout.sch (KiCad schematic (older format))
At the start: 3 parts, among them IC1 MCP6002, P1 CONN_01X04, P2 CONN_01X04

Commit message: Upon fabrication, we have discovered this is not a SOP-8 socket at all.
Parts:
- IC1: footprint Housings_SSOP:MSOP-8_3x3mm_Pitch0.65mm -> sop8:SOP-8
Changed lines of the file:
@@
 LIBS:valves
 LIBS:misc
+LIBS:sop8breakout-cache
 EELAYER 25 0
 EELAYER END
@@
 F 0 "IC1" H 6100 4000 60  0000 C CNN
 F 1 "MCP6002" V 5800 3700 60  0000 C CNN
-F 2 "Housings_SSOP:MSOP-8_3x3mm_Pitch0.65mm" H 5800 3700 60  0001 C CNN
+F 2 "sop8:SOP-8" H 5800 3700 60  0001 C CNN
 F 3 "" H 5800 3700 60  0000 C CNN
 	1    5800 3700
